File: kicad-rs-converter/kicad-rs-converter.kicad_sch (KiCad schematic)
At the start: 29 parts, among them X1 CONN_PWR, X2 CONN_RS232, X3 CONN_2

Commit message: footprints for MAX232 & MAX485
Parts:
- DA1: footprint Package_CDFP_RU:402.16-32 -> Package_SO:SO-16_3.9x9.9mm_P1.27mm
- DA3: footprint Package_CDFP_RU:Н02.8-1В -> Package_SO:SO-8_3.9x4.9mm_P1.27mm
Changed lines of the file:
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@@
 			)
 		)
-		(property "Footprint" "Package_CDFP_RU:402.16-32"
+		(property "Footprint" "Package_SO:SO-16_3.9x9.9mm_P1.27mm"
 			(at 119.38 260.35 0)
 			(effects
@@
 			)
 		)
-		(property "Footprint" "Package_CDFP_RU:Н02.8-1В"
+		(property "Footprint" "Package_SO:SO-8_3.9x4.9mm_P1.27mm"
 			(at 275.59 168.91 0)
 			(effects

Commit message: Placed footprints for LED
Parts:
- HL1, HL2: footprint (none) -> LED_SMD:LED_1210_3225Metric
Changed lines of the file:
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@@
 			)
 		)
-		(property "Footprint" ""
+		(property "Footprint" "LED_SMD:LED_1210_3225Metric"
 			(at 36.83 260.4008 0)
 			(effects
@@
 			)
 		)
-		(property "Footprint" ""
+		(property "Footprint" "LED_SMD:LED_1210_3225Metric"
 			(at 189.23 171.5008 0)
 			(effects

Commit message: Placed footprints for Resistors
Parts:
- R1, R10, R2, R3, R4, R5, R6, R7, R8, R9: footprint (none) -> Resistor_SMD:R_0603_1608Metric
- VD1: footprint (none) -> Diode_SMD:D_0805_2012Metric
Changed lines of the file:
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@@
 			)
 		)
-		(property "Footprint" ""
+		(property "Footprint" "Resistor_SMD:R_0603_1608Metric"
 			(at 321.945 154.94 0)
 			(effects
@@
 			)
 		)
-		(property "Footprint" ""
+		(property "Footprint" "Resistor_SMD:R_0603_1608Metric"
 			(at 307.34 137.795 0)
 			(effects
@@
 			)
 		)
-		(property "Footprint" ""
+		(property "Footprint" "Resistor_SMD:R_0603_1608Metric"
 			(at 251.46 51.435 0)
 			(effects
@@
 			)
 		)
-		(property "Footprint" ""
+		(property "Footprint" "Resistor_SMD:R_0603_1608Metric"
 			(at 226.695 177.8 0)
 			(effects
@@
 			)
 		)
-		(property "Footprint" ""
+		(property "Footprint" "Resistor_SMD:R_0603_1608Metric"
 			(at 188.595 154.94 0)
 			(effects
@@
 			)
 		)
-		(property "Footprint" ""
+		(property "Footprint" "Resistor_SMD:R_0603_1608Metric"
 			(at 36.195 243.84 0)
 			(effects
@@
 			)
 		)
-		(property "Footprint" ""
+		(property "Footprint" "Resistor_SMD:R_0603_1608Metric"
 			(at 334.01 107.315 0)
 			(effects
@@
 			)
 		)
-		(property "Footprint" ""
+		(property "Footprint" "Resistor_SMD:R_0603_1608Metric"
 			(at 196.215 90.17 0)
 			(effects
@@
 			)
 		)
-		(property "Footprint" ""
+		(property "Footprint" "Diode_SMD:D_0805_2012Metric"
 			(at 78.6892 46.99 0)
 			(effects
@@
 			)
 		)
-		(property "Footprint" ""
+		(property "Footprint" "Resistor_SMD:R_0603_1608Metric"
 			(at 203.2 50.165 0)
 			(effects
@@
 			)
 		)
-		(property "Footprint" ""
+		(property "Footprint" "Resistor_SMD:R_0603_1608Metric"
 			(at 344.17 147.955 0)
 			(effects

Commit message: Placed footprints for polar capacitors
Parts:
- C1, C2, C3, C5, C7, C8: footprint (none) -> Capacitor_SMD:CP_Elec_4x5.8
Changed lines of the file:
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@@
 			)
 		)
-		(property "Footprint" ""
+		(property "Footprint" "Capacitor_SMD:CP_Elec_4x5.8"
 			(at 88.265 57.15 0)
 			(effects
@@
 			)
 		)
-		(property "Footprint" ""
+		(property "Footprint" "Capacitor_SMD:CP_Elec_4x5.8"
 			(at 74.93 241.935 0)
 			(effects
@@
 			)
 		)
-		(property "Footprint" ""
+		(property "Footprint" "Capacitor_SMD:CP_Elec_4x5.8"
 			(at 184.15 230.505 0)
 			(effects
@@
 			)
 		)
-		(property "Footprint" ""
+		(property "Footprint" "Capacitor_SMD:CP_Elec_4x5.8"
 			(at 137.795 58.42 0)
 			(effects
@@
 			)
 		)
-		(property "Footprint" ""
+		(property "Footprint" "Capacitor_SMD:CP_Elec_4x5.8"
 			(at 91.44 266.065 0)
 			(effects
@@
 			)
 		)
-		(property "Footprint" ""
+		(property "Footprint" "Capacitor_SMD:CP_Elec_4x5.8"
 			(at 198.755 257.81 0)
 			(effects

Commit message: Footprint for SMD Capacitors and Resistors
Parts:
- C4, C6: footprint (none) -> Capacitor_SMD:C_0805_2012Metric
- R11: footprint (none) -> Resistor_SMD:R_0603_1608Metric
Changed lines of the file:
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@@
 			)
 		)
-		(property "Footprint" ""
+		(property "Footprint" "Resistor_SMD:R_0603_1608Metric"
 			(at 371.475 142.24 0)
 			(effects
@@
 			)
 		)
-		(property "Footprint" ""
+		(property "Footprint" "Capacitor_SMD:C_0805_2012Metric"
 			(at 156.845 69.85 0)
 			(effects
@@
 			)
 		)
-		(property "Footprint" ""
+		(property "Footprint" "Capacitor_SMD:C_0805_2012Metric"
 			(at 103.505 69.85 0)
 			(effects

Commit message: Changed from polar CP capacitors to regular capacitors C
Parts:
- C1, C2, C3, C5, C7, C8: footprint Capacitor_SMD:CP_Elec_4x5.8 -> (none); symbol Device_GOST:CP -> Device_GOST:C
- C4, C6: footprint Capacitor_SMD:C_0805_2012Metric -> (none)
Changed lines of the file:
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@@
 	)
 	(symbol
-		(lib_id "Device_GOST:CP")
+		(lib_id "Device_GOST:C")
 		(at 90.17 57.15 0)
 		(unit 1)
@@
 			)
 		)
-		(property "Footprint" "Capacitor_SMD:CP_Elec_4x5.8"
+		(property "Footprint" ""
 			(at 88.265 57.15 0)
 			(effects
@@
 	)
 	(symbol
-		(lib_id "Device_GOST:CP")
+		(lib_id "Device_GOST:C")
 		(at 74.93 240.03 90)
 		(unit 1)
@@
 			)
 		)
-		(property "Footprint" "Capacitor_SMD:CP_Elec_4x5.8"
+		(property "Footprint" ""
 			(at 74.93 241.935 0)
 			(effects
@@
 	)
 	(symbol
-		(lib_id "Device_GOST:CP")
+		(lib_id "Device_GOST:C")
 		(at 184.15 228.6 90)
 		(unit 1)
@@
 			)
 		)
-		(property "Footprint" "Capacitor_SMD:CP_Elec_4x5.8"
+		(property "Footprint" ""
 			(at 184.15 230.505 0)
 			(effects
@@
 			)
 		)
-		(property "Footprint" "Capacitor_SMD:C_0805_2012Metric"
+		(property "Footprint" ""
 			(at 156.845 69.85 0)
 			(effects
@@
 	)
 	(symbol
-		(lib_id "Device_GOST:CP")
+		(lib_id "Device_GOST:C")
 		(at 139.7 58.42 0)
 		(unit 1)
@@
 			)
 		)
-		(property "Footprint" "Capacitor_SMD:CP_Elec_4x5.8"
+		(property "Footprint" ""
 			(at 137.795 58.42 0)
 			(effects
@@
 	)
 	(symbol
-		(lib_id "Device_GOST:CP")
+		(lib_id "Device_GOST:C")
 		(at 91.44 264.16 90)
 		(unit 1)
@@
 			)
 		)
-		(property "Footprint" "Capacitor_SMD:CP_Elec_4x5.8"
+		(property "Footprint" ""
 			(at 91.44 266.065 0)
 			(effects
@@
 	)
 	(symbol
-		(lib_id "Device_GOST:CP")
+		(lib_id "Device_GOST:C")
 		(at 196.85 257.81 180)
 		(unit 1)
@@
 			)
 		)
-		(property "Footprint" "Capacitor_SMD:CP_Elec_4x5.8"
+		(property "Footprint" ""
 			(at 198.755 257.81 0)
 			(effects
@@
 			)
 		)
-		(property "Footprint" "Capacitor_SMD:C_0805_2012Metric"
+		(property "Footprint" ""
 			(at 103.505 69.85 0)
 			(effects

Commit message: Assigned footprint of SMD:C_1206_3216 Metric to every capacitor
Parts:
- C1, C2, C3, C4, C5, C6, C7, C8: footprint (none) -> Capacitor_SMD:C_1206_3216Metric
Changed lines of the file:
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@@
 			)
 		)
-		(property "Footprint" ""
+		(property "Footprint" "Capacitor_SMD:C_1206_3216Metric"
 			(at 88.265 57.15 0)
 			(effects
@@
 			)
 		)
-		(property "Footprint" ""
+		(property "Footprint" "Capacitor_SMD:C_1206_3216Metric"
 			(at 74.93 241.935 0)
 			(effects
@@
 			)
 		)
-		(property "Footprint" ""
+		(property "Footprint" "Capacitor_SMD:C_1206_3216Metric"
 			(at 184.15 230.505 0)
 			(effects
@@
 			)
 		)
-		(property "Footprint" ""
+		(property "Footprint" "Capacitor_SMD:C_1206_3216Metric"
 			(at 156.845 69.85 0)
 			(effects
@@
 			)
 		)
-		(property "Footprint" ""
+		(property "Footprint" "Capacitor_SMD:C_1206_3216Metric"
 			(at 137.795 58.42 0)
 			(effects
@@
 			)
 		)
-		(property "Footprint" ""
+		(property "Footprint" "Capacitor_SMD:C_1206_3216Metric"
 			(at 91.44 266.065 0)
 			(effects
@@
 			)
 		)
-		(property "Footprint" ""
+		(property "Footprint" "Capacitor_SMD:C_1206_3216Metric"
 			(at 198.755 257.81 0)
 			(effects
@@
 			)
 		)
-		(property "Footprint" ""
+		(property "Footprint" "Capacitor_SMD:C_1206_3216Metric"
 			(at 103.505 69.85 0)
 			(effects

Commit message: Assigned footprints for X connector — Terminal Block
Parts:
- X1, X3: footprint (none) -> TerminalBlock_Phoenix:TerminalBlock_Phoenix_PT-1,5-2-5.0-H_1x02_P5.00mm_Horizontal
- X2: footprint (none) -> TerminalBlock_Phoenix:TerminalBlock_Phoenix_PT-1,5-3-5.0-H_1x03_P5.00mm_Horizontal
Changed lines of the file:
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@@
 			)
 		)
-		(property "Footprint" ""
+		(property "Footprint" "TerminalBlock_Phoenix:TerminalBlock_Phoenix_PT-1,5-2-5.0-H_1x02_P5.00mm_Horizontal"
 			(at 60.96 36.83 0)
 			(effects
@@
 			)
 		)
-		(property "Footprint" ""
+		(property "Footprint" "TerminalBlock_Phoenix:TerminalBlock_Phoenix_PT-1,5-2-5.0-H_1x02_P5.00mm_Horizontal"
 			(at 382.27 162.56 0)
 			(effects
@@
 			)
 		)
-		(property "Footprint" ""
+		(property "Footprint" "TerminalBlock_Phoenix:TerminalBlock_Phoenix_PT-1,5-3-5.0-H_1x03_P5.00mm_Horizontal"
 			(at 137.16 154.94 0)
 			(effects
