File: kicad-rs-converter/kicad-rs-converter.kicad_pcb (KiCad board)
At the start: 2 copper layers, 60 x 40 mm, 29 parts, among them X1 CONN_PWR, X2 CONN_RS232, X3 CONN_2

Commit message: transistor flip and reconnect on pcbdoc
Parts:
- moved R3 3.90 mm to (171.3, 126.8)
- moved VT1 0.34 mm to (167.7, 131.1), turned to -90 degrees
Connections:
- R3 pad 2: Net-(VT1-E) -> Net-(VT1-B)
- R4 pad 1: Net-(VT1-E) -> Net-(VT1-B)
- R6 pad 2: Net-(VT1-E) -> Net-(VT1-B)
- VT1 pad 1: Net-(DA3-DE) -> Net-(VT1-B)
- VT1 pad 2: Net-(VT1-E) -> +5V
- VT1 pad 3: +5V -> Net-(DA3-DE)
Routing:
- net Net-(VT1-B): track 0.00 -> 10.2 mm
- net Net-(VT1-E): track 6.71 -> 0.00 mm
- net Net-(DA1-~{RXOUT1}): track 31.2 -> 28.1 mm
- net Net-(DA3-DE): track 31.7 -> 29.2 mm
- net +5V: track 231.2 -> 230.5 mm
- net Net-(R11-Pad2): track 21.1 -> 21.7 mm
